File: vfd_display.kicad_sch (KiCad schematic)
At the start: 60 parts, among them J1 Conn_01x04, J2 Conn_01x04, J4 PJ-036AH-SMT-TR, Q1 STD16N65M5, U1 LM3478, U2 LR12LG-G, U3 TLP170AM, U5 GP1294AI, U6 TPS56628

Commit message: BOM Update
Parts:
- removed C12: 1uF, Capacitor_SMD:C_0805_2012Metric_Pad1.18x1.45mm_HandSolder, symbol Device:C
- removed C13, C28: 100nF, Capacitor_SMD:C_0805_2012Metric_Pad1.18x1.45mm_HandSolder, symbol Device:C
- removed C14, C26: 10uF, Capacitor_SMD:C_0805_2012Metric_Pad1.18x1.45mm_HandSolder, symbol Device:C
- removed C29: 15pF, Capacitor_SMD:C_0805_2012Metric_Pad1.18x1.45mm_HandSolder, symbol Device:C
- removed C30: 47uF, Capacitor_SMD:C_0805_2012Metric_Pad1.18x1.45mm_HandSolder, symbol Device:C
- removed L2: 2.2uH, Inductor_SMD:L_Bourns_SRR1260, symbol Device:L
- removed R10: 100k, Resistor_SMD:R_0805_2012Metric_Pad1.20x1.40mm_HandSolder, symbol Device:R_US
- removed R11: 10k, Resistor_SMD:R_0805_2012Metric_Pad1.20x1.40mm_HandSolder, symbol Device:R_US
- removed R12: 73k2, Resistor_SMD:R_0805_2012Metric_Pad1.20x1.40mm_HandSolder, symbol Device:R_US
- removed R13: 68R, Resistor_SMD:R_0805_2012Metric_Pad1.20x1.40mm_HandSolder, symbol Device:R_US
- removed R25: 22k1, Resistor_SMD:R_0805_2012Metric_Pad1.20x1.40mm_HandSolder, symbol Device:R_US
- removed U3: TLP170AM, Remi_Footprints:Toshiba-11-4M1S, symbol Remi_Symbols:TLP170AM
- removed U6: TPS56628, Package_SO:SOIC-8_3.9x4.9mm_P1.27mm, symbol Remi_Symbols:TPS56628
- added C20, C22, C3, C5: 100nF, Capacitor_SMD:C_0805_2012Metric_Pad1.18x1.45mm_HandSolder, symbol Device:C
- added C21, C4: 10uF, Capacitor_SMD:C_0805_2012Metric_Pad1.18x1.45mm_HandSolder, symbol Device:C
- added C23, C24, C6, C7: 22uF, Capacitor_SMD:C_0805_2012Metric_Pad1.18x1.45mm_HandSolder, symbol Device:C
- added L1, L3: 2.2 uH, Inductor_SMD:L_1008_2520Metric_Pad1.43x2.20mm_HandSolder, symbol Device:L
- added R19, R3: 31k6, Resistor_SMD:R_0805_2012Metric_Pad1.20x1.40mm_HandSolder, symbol Device:R_US
- added R20, R21, R5: 10k, Resistor_SMD:R_0805_2012Metric_Pad1.20x1.40mm_HandSolder, symbol Device:R_US
- added U2, U5: AP62250WU-7, Remi_Footprints:TSOT26, symbol Regulator_Switching:AP62250Z6
- F1: value MFU0805FF03000P100 -> 3A; DigiKeu (none) -> MFU0805FF03000P100
- J1: footprint Connector_JST:JST_PH_S4B-PH-SM4-TB_1x04-1MP_P2.00mm_Horizontal -> Remi_Footprints:M20-8900405; Digi-Key 455-S4B-PH-SM4-TBCT-ND -> 952-3265-ND
- J2: footprint Connector_JST:JST_PH_S4B-PH-SM4-TB_1x04-1MP_P2.00mm_Horizontal -> Remi_Footprints:M20-8900405; Digi-Key 455-S4B-PH-SM4-TBCT-ND -> M20-8900405
- renumbered C9 to C1, C3 to C10, C1 to C11, C5 to C12, C6 to C13, C7 to C14, C11 to C15, C24 to C16, C25 to C17, C8 to C18, C27 to C19, C10 to C2, C2 to C8, C4 to C9, D8 to D2, D4 to D3, D5 to D4, D6 to D5, D7 to D6, J4 to J3, L1 to L2, R8 to R1, R20 to R10, R2 to R11, R4 to R12, R6 to R13, R1 to R14, R21 to R15, R22 to R16, R23 to R17, R24 to R18, R9 to R2, R7 to R4, R5 to R6, R17 to R7, R3 to R8, R19 to R9, U2 to U1, U5 to U3, U1 to U4
Connections:
- net 12V: now also C21.1, C22.1, C4.1, C5.1, U2.3 (VIN), U5.3 (VIN)
- net FILAMENT_EN: now also R20.2, U5.5 (EN)
- net GND: now also C21.2, C22.2, C23.2, C24.2, C4.2, C5.2, C6.2, C7.2, R20.1, R21.1, R5.1, U2.1 (GND), U5.1 (GND)
- net VDD: now also C6.1, C7.1, L1.2, R3.2
- net V_FILAMENT: now also C23.1, C24.1, L3.2, R19.2
- new net: C20.2, L3.1, U5.2 (SW)
- new net: C3.2, L1.1, U2.2 (SW)
- new net: R3.1, R5.2, U2.4 (FB)
- new net: C3.1, U2.6 (BST)
- new net: C20.1, U5.6 (BST)
- new net: R19.1, R21.2, U5.4 (FB)
- no-connect marks 8 -> 9
Other:
- moved on the sheet: F1, J3

Commit message: Fabrication outputs
Other:
- note added: "github.com/RemiFM/VFD-Power-Supply"
Changed lines of the file:
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@@
     (effects (font (size 2.54 2.54) (thickness 0.254) bold) (justify left bottom))
+  )
+  (text "github.com/RemiFM/VFD-Power-Supply" (at 190.5 177.8 0)
+    (effects (font (face "Comic Sans MS") (size 3 3) (thickness 0.56) bold (color 204 102 0 1)) (justify left bottom) (href "https://github.com/RemiFM/VFD-Power-Supply"))
   )
   (text "VFD DISPLAY" (at 179.07 77.47 0)
