File: vfd_display.kicad_pcb (KiCad board)
At the start: 2 copper layers, 154 x 54 mm, 73 parts, among them J1 Conn_01x04, J2 Conn_01x04, J4 PJ-036AH-SMT-TR, Q1 STD16N65M5, U1 LM3478, U2 LR12LG-G, U3 TLP170AM, U5 GP1294AI, U6 TPS56628

Commit message: BOM Update
Parts:
- removed the C12 at (168.0, 96.0)
- removed the C13 at (147.5, 90.2)
- removed the C14 at (150.5, 90.2)
- removed C26: 10uF, Capacitor_SMD:C_0805_2012Metric_Pad1.18x1.45mm_HandSolder
- removed C28: 100nF, Capacitor_SMD:C_0805_2012Metric_Pad1.18x1.45mm_HandSolder
- removed C29: 15pF, Capacitor_SMD:C_0805_2012Metric_Pad1.18x1.45mm_HandSolder
- removed C30: 47uF, Capacitor_SMD:C_0805_2012Metric_Pad1.18x1.45mm_HandSolder
- removed the G*** at (198.0, 88.0)
- removed the GND at (144.5, 86.5)
- removed the L2 at (180.0, 93.5)
- removed the R10 at (165.0, 96.0)
- removed the R11 at (159.5, 89.0)
- removed the R12 at (168.5, 89.0)
- removed the R13 at (213.5, 75.8)
- removed R25: 22k1, Resistor_SMD:R_0805_2012Metric_Pad1.20x1.40mm_HandSolder
- removed the U3 at (216.0, 70.5)
- removed U6: TPS56628, Package_SO:SOIC-8_3.9x4.9mm_P1.27mm
- added C20: 100nF, Capacitor_SMD:C_0805_2012Metric_Pad1.18x1.45mm_HandSolder, B.Cu at (167.5, 103.9)
- added C21: 10uF, Capacitor_SMD:C_0805_2012Metric_Pad1.18x1.45mm_HandSolder, B.Cu at (157.8, 99.9)
- added C22: 100nF, Capacitor_SMD:C_0805_2012Metric_Pad1.18x1.45mm_HandSolder, B.Cu at (160.2, 99.9)
- added C23: 22uF, Capacitor_SMD:C_0805_2012Metric_Pad1.18x1.45mm_HandSolder, B.Cu at (160.2, 103.9)
- added C24: 22uF, Capacitor_SMD:C_0805_2012Metric_Pad1.18x1.45mm_HandSolder, B.Cu at (157.8, 103.9)
- added C3: 100nF, Capacitor_SMD:C_0805_2012Metric_Pad1.18x1.45mm_HandSolder, B.Cu at (165.0, 83.0)
- added C4: 10uF, Capacitor_SMD:C_0805_2012Metric_Pad1.18x1.45mm_HandSolder, B.Cu at (161.0, 90.3)
- added C5: 100nF, Capacitor_SMD:C_0805_2012Metric_Pad1.18x1.45mm_HandSolder, B.Cu at (161.0, 92.8)
- added C6: 22uF, Capacitor_SMD:C_0805_2012Metric_Pad1.18x1.45mm_HandSolder, B.Cu at (165.0, 92.8)
- added C7: 22uF, Capacitor_SMD:C_0805_2012Metric_Pad1.18x1.45mm_HandSolder, B.Cu at (165.0, 90.3)
- added G***: LOGO, LOGO, F.Cu at (151.0, 90.5)
- added G***: LOGO, LOGO, B.Cu at (196.0, 90.0)
- added G***: LOGO, LOGO, B.Cu at (179.5, 97.0)
- added L1: 2.2 uH, Inductor_SMD:L_1008_2520Metric_Pad1.43x2.20mm_HandSolder, B.Cu at (166.0, 86.7)
- added L3: 2.2 uH, Inductor_SMD:L_1008_2520Metric_Pad1.43x2.20mm_HandSolder, B.Cu at (164.0, 105.0)
- added R19: 31k6, Resistor_SMD:R_0805_2012Metric_Pad1.20x1.40mm_HandSolder, B.Cu at (167.6, 99.0)
- added R20: 10k, Resistor_SMD:R_0805_2012Metric_Pad1.20x1.40mm_HandSolder, B.Cu at (170.6, 102.0)
- added R21: 10k, Resistor_SMD:R_0805_2012Metric_Pad1.20x1.40mm_HandSolder, B.Cu at (164.0, 98.5)
- added R3: 31k6, Resistor_SMD:R_0805_2012Metric_Pad1.20x1.40mm_HandSolder, B.Cu at (161.5, 82.5)
- added R5: 10k, Resistor_SMD:R_0805_2012Metric_Pad1.20x1.40mm_HandSolder, B.Cu at (159.5, 86.5)
- added REF**: Polarity_Center_Positive_6mm_SilkScreen, Symbol:Polarity_Center_Positive_6mm_SilkScreen, B.Cu at (82.5, 90.0)
- added U2: AP62250WU-7, Remi_Footprints:TSOT26, B.Cu at (162.6, 86.6)
- added U5: AP62250WU-7, Remi_Footprints:TSOT26, B.Cu at (164.0, 101.5)
- F1: value MFU0805FF03000P100 -> 4A
- J1, J2: footprint Connector_JST:JST_PH_S4B-PH-SM4-TB_1x04-1MP_P2.00mm_Horizontal -> Remi_Footprints:M20-8900405
- moved J2 7.21 mm to (214.0, 98.0)
- moved J1 7.17 mm to (214.0, 82.4)
- renumbered C9 to C1, C3 to C10, C1 to C11, C5 to C12, C6 to C13, C7 to C14, C11 to C15, C24 to C16, C25 to C17, C8 to C18, C27 to C19, C10 to C2, C2 to C8, C4 to C9, D8 to D2, D4 to D3, D5 to D4, D6 to D5, D7 to D6, J4 to J3, L1 to L2, R8 to R1, R20 to R10, R2 to R11, R4 to R12, R6 to R13, R1 to R14, R21 to R15, R22 to R16, R23 to R17, R24 to R18, R9 to R2, R7 to R4, R5 to R6, R17 to R7, R3 to R8, R19 to R9, U2 to U1, U5 to U3, U1 to U4
Routing:
- net VDD: track 132.6 -> 49.6 mm, vias 0 -> 2
- net GND: track 157.1 -> 92.5 mm, vias 20 -> 97
- net Net-(U6-SW): track 29.3 -> 0.00 mm
- net FILAMENT_EN: track 29.1 -> 49.3 mm
- net V_FILAMENT: track 11.5 -> 22.7 mm, vias 0 -> 2
- net Net-(U6-VFB): track 9.55 -> 0.00 mm
- net Net-(U6-VREG): track 6.04 -> 0.00 mm
- net Net-(U5-FB): track 0.00 -> 5.89 mm
- net VFD_RESET: track 27.0 -> 22.5 mm
- net VFD_SDA: track 30.2 -> 25.7 mm
- net Net-(U2-FB): track 0.00 -> 4.15 mm
- net 12V: track 66.9 -> 71.0 mm
- net Net-(U6-EN): track 4.07 -> 0.00 mm
- net VFD_CS: track 33.0 -> 28.9 mm
- net VFD_SCK: track 35.8 -> 32.1 mm
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- added copper zone on B.Cu, net Net-(D2-K)
- added copper zone on B.Cu, net Net-(U2-SW)
- added copper zone on B.Cu, net Net-(U5-FB)
- added copper zone on B.Cu, net Net-(U5-SW)
- added copper zone on B.Cu, net V_FILAMENT
Other:
- board text added: "12V INPUT"

Commit message: Fabrication outputs
Parts:
- added G***: LOGO, LOGO, F.Cu at (151.0, 90.5)

Commit message: Minor tweaks
Routing:
- net GND: vias 97 -> 101

Commit message: GP1278BI Variation
Parts:
- U3: footprint Remi_Footprints:VFD_GP1294AI -> Remi_Footprints:VFD_GP1287BI
Routing:
- net Net-(U3-VHP): track 4.50 -> 7.27 mm
